Commit message: Update button.xacro

File: UR3_sim/ur3_sim_description/urdf/button.xacro (robot description, xacro)
@@ -23,5 +23,5 @@
       <origin xyz="0.477 0.1 0.42" rpy="1.5707 0.0 -1.5707"/>
     </joint>
-     <link name="button2">
+    <!-- <link name="button2">
       <visual>
        <geometry>
@@ -29,9 +29,9 @@
         </geometry>
       </visual>
-     <!-- <collision>
+      <collision>
        <geometry>
           <mesh filename="package://ur3_sim_description/meshes/button/ERC2022_button_ID1.dae" scale="0.001 0.001 0.001"/>
         </geometry>
-      </collision> -->
+      </collision>
       <inertial>
         <mass value="10" />
@@ -43,16 +43,16 @@
       <child link="button2"/>
       <origin xyz="0.477 0 0.42" rpy="1.5707 0.0 -1.5707"/>
-    </joint>
-    <link name="button3">
+    </joint>-->
+ <!--   <link name="button3">
       <visual>
+        <geometry>
+          <mesh filename="package://ur3_sim_description/meshes/button/ERC2022_button_ID3.dae" scale="0.001 0.001 0.001"/>
+        </geometry>
+      </visual>
+      <collision>
         <geometry>
           <mesh filename="package://ur3_sim_description/meshes/button/ERC2022_button_ID2.dae" scale="0.001 0.001 0.001"/>
         </geometry>
-      </visual>
-    <!--  <collision>
-        <geometry>
-          <mesh filename="package://ur3_sim_description/meshes/button/ERC2022_button_ID2.dae" scale="0.001 0.001 0.001"/>
-        </geometry>
-      </collision>-->
+      </collision>
       <inertial>
         <mass value="10" />
@@ -64,6 +64,6 @@
       <child link="button3"/>
       <origin xyz="0.477 -0.1 0.42" rpy="1.5707 0.0 -1.5707"/>
-    </joint>
- <link name="button4">
+    </joint>-->
+<!-- <link name="button4">
       <visual>
        <geometry>
@@ -71,9 +71,9 @@
         </geometry>
       </visual>
-      <!-- <collision>
+       <collision>
        <geometry>
           <mesh filename="package://ur3_sim_description/meshes/button/ERC2022_button_ID1.dae" scale="0.001 0.001 0.001"/>
         </geometry>
-      </collision> -->
+      </collision>
       <inertial>
         <mass value="10" />
@@ -85,5 +85,5 @@
       <child link="button4"/>
       <origin xyz="0.477 0.1 0.26" rpy="1.5707 0.0 -1.5707"/>
-    </joint>
+    </joint> -->
     <link name="button5">
       <visual>
@@ -110,5 +110,5 @@
       <visual>
         <geometry>
-          <mesh filename="package://ur3_sim_description/meshes/button/ERC2022_button_ID1.dae" scale="0.001 0.001 0.001"/>
+          <mesh filename="package://ur3_sim_description/meshes/button/ERC2022_button_ID3.dae" scale="0.001 0.001 0.001"/>
         </geometry>
       </visual>
@@ -128,15 +128,15 @@
       <origin xyz="0.477 -0.1 0.26" rpy="1.5707 0.0 -1.5707"/>
     </joint>
-    <link name="button7">
+  <!--  <link name="button7">
       <visual>
         <geometry>
-          <mesh filename="package://ur3_sim_description/meshes/button/ERC2022_button_ID2.dae" scale="0.001 0.001 0.001"/>
+          <mesh filename="package://ur3_sim_description/meshes/button/ERC2022_button_ID7.dae" scale="0.001 0.001 0.001"/>
         </geometry>
       </visual>
-   <!--  <collision>
+     <collision>
         <geometry>
           <mesh filename="package://ur3_sim_description/meshes/button/ERC2022_button_ID3.dae" scale="0.001 0.001 0.001"/>
         </geometry>
-      </collision>-->
+      </collision>
       <inertial>
         <mass value="10" />
@@ -148,16 +148,16 @@
       <child link="button7"/>
       <origin xyz="0.477 0.1 0.1" rpy="1.5707 0.0 -1.5707"/>
-    </joint>
- <link name="button8">
+    </joint>-->
+ <!-- <link name="button8">
       <visual>
+        <geometry>
+          <mesh filename="package://ur3_sim_description/meshes/button/ERC2022_button_ID8.dae" scale="0.001 0.001 0.001"/>
+        </geometry>
+      </visual>
+    <collision>
         <geometry>
           <mesh filename="package://ur3_sim_description/meshes/button/ERC2022_button_ID4.dae" scale="0.001 0.001 0.001"/>
         </geometry>
-      </visual>
-   <!--  <collision>
-        <geometry>
-          <mesh filename="package://ur3_sim_description/meshes/button/ERC2022_button_ID4.dae" scale="0.001 0.001 0.001"/>
-        </geometry>
-      </collision> -->
+      </collision>
       <inertial>
         <mass value="10" />
@@ -169,9 +169,9 @@
       <child link="button8"/>
       <origin xyz="0.477 0 0.1" rpy="1.5707 0.0 -1.5707"/>
-    </joint>
+    </joint>-->
     <link name="button9">
       <visual>
         <geometry>
-          <mesh filename="package://ur3_sim_description/meshes/button/ERC2022_button_ID3.dae" scale="0.001 0.001 0.001"/>
+          <mesh filename="package://ur3_sim_description/meshes/button/ERC2022_button_ID4.dae" scale="0.001 0.001 0.001"/>
         </geometry>
       </visual>
