Commit message: Cell Pushed back

File: UR3_sim/ur3_sim_description/urdf/box.xacro (robot description, xacro)
@@ -21,5 +21,5 @@
       <parent link="base_link"/>
       <child link="box_bottom"/>
-      <origin xyz="0.3816 -0.29 0.17" rpy="0.0 0.0 -1.8849555922"/>
+      <origin xyz="0.5016 -0.29 0.17" rpy="0.0 0.0 -1.8849555922"/>
     </joint>
     <link name="box_top">
@@ -42,5 +42,6 @@
       <parent link="base_link"/>
       <child link="box_top"/>
-      <origin xyz="0.3816 -0.29 0.17" rpy="0.0 0.0 -1.8849555922"/>
+      <!-- <origin xyz="0.3816 -0.29 0.17" rpy="0.0 0.0 -1.8849555922"/> -->
+      <origin xyz="0.29 -0.25 -0.2" rpy="0.0 0.0 -1.8849555922"/>
     </joint>
   </xacro:macro>

File: UR3_sim/ur3_sim_description/urdf/button.xacro (robot description, xacro)
@@ -4,10 +4,10 @@
     <link name="button1">
       <visual>
-       <geometry>
+        <geometry>
           <mesh filename="package://ur3_sim_description/meshes/button/ERC2022_button_ID1.dae" scale="0.001 0.001 0.001"/>
         </geometry>
       </visual>
-    <!--   <collision>
-       <geometry>
+      <!-- <collision>
+        <geometry>
           <mesh filename="package://ur3_sim_description/meshes/button/ERC2022_button_ID1.dae" scale="0.001 0.001 0.001"/>
         </geometry>
@@ -21,17 +21,17 @@
       <parent link="base_link"/>
       <child link="button1"/>
-      <origin xyz="0.477 0.1 0.42" rpy="1.5707 0.0 -1.5707"/>
+      <origin xyz="0.597 0.06 0.35" rpy="1.5707 0.0 -1.5707"/>
     </joint>
-    <!-- <link name="button2">
+    <link name="button2">
       <visual>
-       <geometry>
+        <geometry>
           <mesh filename="package://ur3_sim_description/meshes/button/ERC2022_button_ID2.dae" scale="0.001 0.001 0.001"/>
         </geometry>
       </visual>
-      <collision>
-       <geometry>
-          <mesh filename="package://ur3_sim_description/meshes/button/ERC2022_button_ID1.dae" scale="0.001 0.001 0.001"/>
+      <!-- <collision>
+        <geometry>
+          <mesh filename="package://ur3_sim_description/meshes/button/ERC2022_button_ID2.dae" scale="0.001 0.001 0.001"/>
         </geometry>
-      </collision>
+      </collision> -->
       <inertial>
         <mass value="10" />
@@ -42,7 +42,7 @@
       <parent link="base_link"/>
       <child link="button2"/>
-      <origin xyz="0.477 0 0.42" rpy="1.5707 0.0 -1.5707"/>
-    </joint>-->
- <!--   <link name="button3">
+      <origin xyz="0.597 -0.06 0.35" rpy="1.5707 0.0 -1.5707"/>
+    </joint>
+    <link name="button3">
       <visual>
         <geometry>
@@ -50,9 +50,9 @@
         </geometry>
       </visual>
-      <collision>
+      <!-- <collision>
         <geometry>
-          <mesh filename="package://ur3_sim_description/meshes/button/ERC2022_button_ID2.dae" scale="0.001 0.001 0.001"/>
+          <mesh filename="package://ur3_sim_description/meshes/button/ERC2022_button_ID3.dae" scale="0.001 0.001 0.001"/>
         </geometry>
-      </collision>
+      </collision> -->
       <inertial>
         <mass value="10" />
@@ -63,17 +63,17 @@
       <parent link="base_link"/>
       <child link="button3"/>
-      <origin xyz="0.477 -0.1 0.42" rpy="1.5707 0.0 -1.5707"/>
-    </joint>-->
-<!-- <link name="button4">
+      <origin xyz="0.597 0.06 0.17" rpy="1.5707 0.0 -1.5707"/>
+    </joint>
+    <link name="button4">
       <visual>
-       <geometry>
+        <geometry>
           <mesh filename="package://ur3_sim_description/meshes/button/ERC2022_button_ID4.dae" scale="0.001 0.001 0.001"/>
         </geometry>
       </visual>
-       <collision>
-       <geometry>
-          <mesh filename="package://ur3_sim_description/meshes/button/ERC2022_button_ID1.dae" scale="0.001 0.001 0.001"/>
+      <!-- <collision>
+        <geometry>
+          <mesh filename="package://ur3_sim_description/meshes/button/ERC2022_button_ID4.dae" scale="0.001 0.001 0.001"/>
         </geometry>
-      </collision>
+      </collision> -->
       <inertial>
         <mass value="10" />
@@ -84,110 +84,5 @@
       <parent link="base_link"/>
       <child link="button4"/>
-      <origin xyz="0.477 0.1 0.26" rpy="1.5707 0.0 -1.5707"/>
-    </joint> -->
-    <link name="button5">
-      <visual>
-       <geometry>
-          <mesh filename="package://ur3_sim_description/meshes/button/ERC2022_button_ID2.dae" scale="0.001 0.001 0.001"/>
-        </geometry>
-      </visual>
-    <!--  <collision>
-       <geometry>
-          <mesh filename="package://ur3_sim_description/meshes/button/ERC2022_button_ID1.dae" scale="0.001 0.001 0.001"/>
-        </geometry>
-      </collision> -->
-      <inertial>
-        <mass value="10" />
-        <inertia ixx="1.0" ixy="0.0" ixz="0.0" iyy="1.0" iyz="0.0" izz="1.0" />
-      </inertial>
-    </link>
-    <joint name="button5_joint" type="fixed">
-      <parent link="base_link"/>
-      <child link="button5"/>
-      <origin xyz="0.477 0 0.26" rpy="1.5707 0.0 -1.5707"/>
-    </joint>
-    <link name="button6">
-      <visual>
-        <geometry>
-          <mesh filename="package://ur3_sim_description/meshes/button/ERC2022_button_ID3.dae" scale="0.001 0.001 0.001"/>
-        </geometry>
-      </visual>
-      <!--<collision>
-        <geometry>
-          <mesh filename="package://ur3_sim_description/meshes/button/ERC2022_button_ID2.dae" scale="0.001 0.001 0.001"/>
-        </geometry>
-      </collision>-->
-      <inertial>
-        <mass value="10" />
-        <inertia ixx="1.0" ixy="0.0" ixz="0.0" iyy="1.0" iyz="0.0" izz="1.0" />
-      </inertial>
-    </link>
-    <joint name="button6_joint" type="fixed">
-      <parent link="base_link"/>
-      <child link="button6"/>
-      <origin xyz="0.477 -0.1 0.26" rpy="1.5707 0.0 -1.5707"/>
-    </joint>
-  <!--  <link name="button7">
-      <visual>
-        <geometry>
-          <mesh filename="package://ur3_sim_description/meshes/button/ERC2022_button_ID7.dae" scale="0.001 0.001 0.001"/>
-        </geometry>
-      </visual>
-     <collision>
-        <geometry>
-          <mesh filename="package://ur3_sim_description/meshes/button/ERC2022_button_ID3.dae" scale="0.001 0.001 0.001"/>
-        </geometry>
-      </collision>
-      <inertial>
-        <mass value="10" />
-        <inertia ixx="1.0" ixy="0.0" ixz="0.0" iyy="1.0" iyz="0.0" izz="1.0" />
-      </inertial>
-    </link>
-    <joint name="button7_joint" type="fixed">
-      <parent link="base_link"/>
-      <child link="button7"/>
-      <origin xyz="0.477 0.1 0.1" rpy="1.5707 0.0 -1.5707"/>
-    </joint>-->
- <!-- <link name="button8">
-      <visual>
-        <geometry>
-          <mesh filename="package://ur3_sim_description/meshes/button/ERC2022_button_ID8.dae" scale="0.001 0.001 0.001"/>
-        </geometry>
-      </visual>
-    <collision>
-        <geometry>
-          <mesh filename="package://ur3_sim_description/meshes/button/ERC2022_button_ID4.dae" scale="0.001 0.001 0.001"/>
-        </geometry>
-      </collision>
-      <inertial>
-        <mass value="10" />
-        <inertia ixx="1.0" ixy="0.0" ixz="0.0" iyy="1.0" iyz="0.0" izz="1.0" />
-      </inertial>
-    </link>
-    <joint name="button8_joint" type="fixed">
-      <parent link="base_link"/>
-      <child link="button8"/>
-      <origin xyz="0.477 0 0.1" rpy="1.5707 0.0 -1.5707"/>
-    </joint>-->
-    <link name="button9">
-      <visual>
-        <geometry>
-          <mesh filename="package://ur3_sim_description/meshes/button/ERC2022_button_ID4.dae" scale="0.001 0.001 0.001"/>
-        </geometry>
-      </visual>
-    <!-- <collision>
-        <geometry>
-          <mesh filename="package://ur3_sim_description/meshes/button/ERC2022_button_ID4.dae" scale="0.001 0.001 0.001"/>
-        </geometry>
-      </collision>-->
-      <inertial>
-        <mass value="10" />
-        <inertia ixx="1.0" ixy="0.0" ixz="0.0" iyy="1.0" iyz="0.0" izz="1.0" />
-      </inertial>
-    </link>
-    <joint name="button9_joint" type="fixed">
-      <parent link="base_link"/>
-      <child link="button9"/>
-      <origin xyz="0.477 -0.1 0.1" rpy="1.5707 0.0 -1.5707"/>
+      <origin xyz="0.597 -0.06 0.17" rpy="1.5707 0.0 -1.5707"/>
     </joint>
   </xacro:macro>

File: UR3_sim/ur3_sim_description/urdf/cell.xacro (robot description, xacro)
@@ -8,9 +8,9 @@
         </geometry>
       </visual>
-  <!--    <collision>
+      <!-- <collision>
         <geometry>
           <mesh filename="package://ur3_sim_description/meshes/cell/ERC2022_cela_white.dae" scale="0.001 0.001 0.001"/>
         </geometry>
-      </collision>-->
+      </collision> -->
       <inertial>
         <mass value="10" />
@@ -21,5 +21,6 @@
       <parent link="world"/>
       <child link="cela_white"/>
-      <origin xyz="-0.04 0.0 -0.14" rpy="0.0 0 -1.57079632679"/>
+      <origin xyz="0.08 0.0 -0.14" rpy="0.0 0 -1.57079632679"/>
+      <!-- <origin xyz="-0.04 0.0 -0.14" rpy="0.0 0 -1.57079632679"/> -->
     </joint>
     <gazebo reference="cela_white">
@@ -32,9 +33,9 @@
         </geometry>
       </visual>
-      <collision>
+      <!-- <collision>
         <geometry>
           <mesh filename="package://ur3_sim_description/meshes/cell/ERC2022_cela_black.dae" scale="0.001 0.001 0.001"/>
         </geometry>
-      </collision>
+      </collision> -->
       <inertial>
         <mass value="10" />
@@ -45,5 +46,5 @@
       <parent link="world"/>
       <child link="cela_black"/>
-      <origin xyz="-0.04 0.0 -0.14" rpy="0.0 0 -1.57079632679"/>
+      <origin xyz="0.08 0.0 -0.14" rpy="0.0 0 -1.57079632679"/>
     </joint>
     <gazebo reference="cela_black">

File: UR3_sim/ur3_sim_description/urdf/gripper.xacro (robot description, xacro)
@@ -18,9 +18,9 @@
         </geometry>
       </visual>
-    <!--   <collision>
+      <collision>
         <geometry>
           <mesh filename="package://ur3_sim_description/meshes/gripper/BaseBottom.dae" scale="0.001 0.001 0.001"/>
         </geometry>
-      </collision>-->
+      </collision>
       <inertial>
         <mass value="0.00002265" />
@@ -41,9 +41,9 @@
         </geometry>
       </visual>
-    <!--  <collision>
+      <collision>
         <geometry>
           <mesh filename="package://ur3_sim_description/meshes/gripper/Adapter.dae" scale="0.001 0.001 0.001"/>
         </geometry>
-      </collision>-->
+      </collision>
       <inertial>
         <mass value="0.00002265" />
@@ -70,10 +70,10 @@
         </geometry>
       </visual>
-    <!-- <collision>
+      <collision>
         <origin xyz="0.0 0 0.0"/>
         <geometry>
           <mesh filename="package://ur3_sim_description/meshes/gripper/MainGear2.dae" scale="0.001 0.001 0.001"/>
         </geometry>
-      </collision>-->
+      </collision>
       <inertial>
         <mass value="0.00002265" />
@@ -103,10 +103,10 @@
         </geometry>
       </visual>
-   <!--  <collision>
+      <collision>
         <origin xyz="-0.044341 0 0.0"/>
         <geometry>
           <mesh filename="package://ur3_sim_description/meshes/gripper/MainGear1.dae" scale="0.001 0.001 0.001"/>
         </geometry>
-      </collision>-->
+      </collision>
       <inertial>
         <mass value="0.00002265" />
@@ -137,10 +137,10 @@
         </geometry>
       </visual>
-   <!--   <collision>
+      <collision>
         <origin xyz="-0.094414 0 0.0"/>
         <geometry>
           <mesh filename="package://ur3_sim_description/meshes/gripper/Arm_R_Bottom.dae" scale="0.001 0.001 0.001"/>
         </geometry>
-      </collision>-->
+      </collision>
       <inertial>
           <mass value="0.0001"/>
@@ -168,10 +168,10 @@
         </geometry>
       </visual>
-  <!--   <collision>
+      <collision>
         <origin xyz="0.050137 0 0.0"/>
         <geometry>
           <mesh filename="package://ur3_sim_description/meshes/gripper/Arm_L_Bottom.dae" scale="0.001 0.001 0.001"/>
         </geometry>
-      </collision>-->
+      </collision>
       <inertial>
           <mass value="0.0001"/>
@@ -199,10 +199,10 @@
         </geometry>
       </visual>
-   <!--  <collision>
+      <collision>
         <origin xyz="0.060137  0 0.027123" rpy="0.0 0.0 0.0"/>
         <geometry>
           <mesh filename="package://ur3_sim_description/meshes/gripper/Arm_R_Top.dae" scale="0.001 0.001 0.001"/>
         </geometry>
-      </collision>-->
+      </collision>
       <inertial>
           <mass value="0.0001"/>
@@ -229,10 +229,10 @@
         </geometry>
       </visual>
-  <!--   <collision>
+      <collision>
         <origin xyz="0.050137 0 0.0"/>
         <geometry>
           <mesh filename="package://ur3_sim_description/meshes/gripper/Arm_L_Top.dae" scale="0.001 0.001 0.001"/>
         </geometry>
-      </collision>-->
+      </collision>
       <inertial>
           <mass value="0.0001"/>
@@ -258,9 +258,9 @@
         </geometry>
       </visual>
-   <!--   <collision>
+      <collision>
         <geometry>
           <mesh filename="package://ur3_sim_description/meshes/gripper/Sock1.dae" scale="0.001 0.001 0.001"/>
         </geometry>
-      </collision>-->
+      </collision>
       <inertial>
         <mass value="0.0000002265" />
@@ -288,9 +288,9 @@
         </geometry>
       </visual>
-  <!--    <collision>
+      <collision>
         <geometry>
           <mesh filename="package://ur3_sim_description/meshes/gripper/Sock2.dae" scale="0.001 0.001 0.001"/>
         </geometry>
-      </collision>-->
+      </collision>
       <inertial>
         <mass value="0.0000002265" />
@@ -317,10 +317,10 @@
         </geometry>
       </visual>
-   <!--  <collision>
+      <collision>
         <origin xyz="-0.01 -0.033 0.0"/>
         <geometry>
           <mesh filename="package://ur3_sim_description/meshes/gripper/Stick1.dae" scale="0.001 0.001 0.001"/>
         </geometry>
-      </collision>-->
+      </collision>
       <inertial>
         <mass value="0.00002265" />
@@ -351,10 +351,10 @@
         </geometry>
       </visual>
-  <!--   <collision>
+      <collision>
         <origin xyz="-0.034341 -0.033 0.0"/>
         <geometry>
           <mesh filename="package://ur3_sim_description/meshes/gripper/Stick2.dae" scale="0.001 0.001 0.001"/>
         </geometry>
-      </collision>-->
+      </collision>
       <inertial>
         <mass value="0.00002265" />
@@ -384,9 +384,9 @@
         </geometry>
       </visual>
-  <!--    <collision>
+      <collision>
         <geometry>
           <mesh filename="package://ur3_sim_description/meshes/gripper/Spacer.dae" scale="0.001 0.001 0.001"/>
         </geometry>
-      </collision>-->
+      </collision>
       <inertial>
         <mass value="0.00002265" />
@@ -414,10 +414,10 @@
         </geometry>
       </visual>
-   <!--   <collision>
+      <collision>
         <origin xyz="-0.01 -0.033 0.0"/>
         <geometry>
           <mesh filename="package://ur3_sim_description/meshes/gripper/Stick_Top1.dae" scale="0.001 0.001 0.001"/>
         </geometry>
-      </collision>-->
+      </collision>
       <inertial>
         <mass value="0.00002265" />
@@ -448,10 +448,10 @@
         </geometry>
       </visual>
-   <!--   <collision>
+      <collision>
         <origin xyz="-0.034341 -0.033 0.0"/>
         <geometry>
           <mesh filename="package://ur3_sim_description/meshes/gripper/Stick_Top2.dae" scale="0.001 0.001 0.001"/>
         </geometry>
-      </collision>-->
+      </collision>
       <inertial>
         <mass value="0.00002265" />
@@ -481,9 +481,9 @@
         </geometry>
       </visual>
-    <!-- <collision>
+      <collision>
         <geometry>
           <mesh filename="package://ur3_sim_description/meshes/gripper/BaseTopCamera.dae" scale="0.001 0.001 0.001"/>
         </geometry>
-      </collision>-->
+      </collision>
       <inertial>
         <mass value="0.00002265" />
@@ -513,9 +513,9 @@
         </geometry>
       </visual>
-   <!--   <collision>
+      <collision>
         <geometry>
           <mesh filename="package://ur3_sim_description/meshes/gripper/CableBlock.dae" scale="0.001 0.001 0.001"/>
         </geometry>
-      </collision>-->
+      </collision>
     </link>
     <joint name="cable_block_joint" type="fixed">

File: UR3_sim/ur3_sim_description/urdf/imu.xacro (robot description, xacro)
@@ -9,10 +9,10 @@
         </geometry>
       </visual>
-    <collision>
+      <!--collision>
         <origin rpy="1.57075 1.57075 -3.1415" xyz="0 -0.025 0"/>
         <geometry>
           <mesh filename="package://ur3_sim_description/meshes/imu/ERC2022_IMU.dae" scale="0.001 0.001 0.001"/>
         </geometry>
-      </collision>
+      </collision>-->
       <inertial>
         <mass value="10" />
@@ -23,5 +23,5 @@
       <parent link="base_link"/>
       <child link="imu"/>
-      <origin rpy="1.57075 0 0" xyz="0.19 0.26 -0.115"/>
+      <origin rpy="1.57075 0 0" xyz="0.31 0.26 -0.115"/>
     </joint>
     <link name="imu_panel"/>
